Commit message: Updated collision definitions in jethexa_description.urdf.xacro to include specific names for coxa, femur, and tibia collisions, enhancing clarity and organization in the URDF structure.

File: jethexa_description/urdf/jethexa_description.urdf.xacro (robot description, xacro)
@@ -46,8 +46,8 @@
                 </material>
             </visual>
-            <collision>
+            <collision name="coxa_collision_${side}${position}">
                 <origin xyz="0.02 0.0 0.0" rpy="0.0 ${my_pi/2} 0.0" />
                 <geometry>
-		    <cylinder radius="0.01" length="${coxa_length}"/>
+		            <cylinder radius="0.01" length="${coxa_length}"/>
                 </geometry>
             </collision>
@@ -77,8 +77,8 @@
                 </material>
             </visual>
-            <collision>
+            <collision name="femur_collision_${side}${position}">
                 <origin xyz="${femur_length/2} 0.0 0.0" rpy="0.0 ${my_pi/2} 0.0" />
                 <geometry>
-		    <cylinder radius="0.01" length="${femur_length}"/>
+		            <cylinder radius="0.01" length="${femur_length}"/>
                 </geometry>
             </collision>
@@ -112,5 +112,5 @@
                 <origin xyz="${tibia_length/2} 0.0 0.0" rpy="0.0 ${my_pi/2} 0.0"/>
                 <geometry>
-		    <cylinder radius="0.01" length="${tibia_length}"/>
+		            <cylinder radius="0.01" length="${tibia_length}"/>
                 </geometry>
             </collision>
